Commit message: Update allegro_hand_description_right.urdf

File: ros2_source/src/allegro_hand_description/urdf/allegro_hand_description_right.urdf (robot description, URDF)
Before this commit: robot allegro_hand_right, 21 links, 20 joints
Links:
- added link wrist
Joints:
- added joint wrist_joint: type fixed, parent palm_link, child wrist, origin xyz=0 0 -0.095 rpy=0 0 0
