Commit message: update right and left urdf

File: ros2_source/src/allegro_hand_description/urdf/allegro_hand_description_left.urdf (robot description, URDF)
Before this commit: robot allegro_hand_left, 21 links, 20 joints
Links:
- added link wrist
- link link_12: geometry collision box size=0.0358 0.034 0.0455; visual mesh filename=package://allegro_hand_description/meshes/link_12.0_left.obj
Joints:
- added joint wrist_joint: type fixed, parent palm_link, child wrist, origin xyz=0 0 -0.095 rpy=0 0 0

File: ros2_source/src/allegro_hand_description/urdf/allegro_hand_description_right.urdf (robot description, URDF)
Before this commit: robot allegro_hand_right, 21 links, 20 joints
Links:
- added link wrist
Joints:
- added joint wrist_joint: type fixed, parent palm_link, child wrist, origin xyz=0 0 -0.095 rpy=0 0 0

Commit message: add allegro_ prefix in urdf

File: ros2_source/src/allegro_hand_description/urdf/allegro_hand_description_left.urdf (robot description, URDF)
Before this commit: robot allegro_hand_left, 22 links, 21 joints
Joints:
- removed joint joint_0
- removed joint joint_1
- removed joint joint_10
- removed joint joint_11
- removed joint joint_11_tip
- removed joint joint_12
- removed joint joint_13
- removed joint joint_14
- removed joint joint_15
- removed joint joint_15_tip
- removed joint joint_2
- removed joint joint_3
- removed joint joint_3_tip
- removed joint joint_4
- removed joint joint_5
- removed joint joint_6
- removed joint joint_7
- removed joint joint_7_tip
- removed joint joint_8
- removed joint joint_9
- added joint allegro_joint_0: type revolute, parent palm_link, child link_0, origin xyz=0 -0.0435 -0.001542 rpy=0.08726646254999999 0 0, axis 0 0 1, limit lower=-0.47 upper=0.47 effort=15 velocity=7
- added joint allegro_joint_1: type revolute, parent link_0, child link_1, origin xyz=0 0 0.0164, axis 0 1 0, limit lower=-0.19599999999999998 upper=1.6099999999999999 effort=15 velocity=7
- added joint allegro_joint_10: type revolute, parent link_9, child link_10, origin xyz=0 0 0.054, axis 0 1 0, limit lower=-0.17400000000000002 upper=1.7089999999999999 effort=15 velocity=7
- added joint allegro_joint_11: type revolute, parent link_10, child link_11, origin xyz=0 0 0.0384, axis 0 1 0, limit lower=-0.227 upper=1.6179999999999999 effort=15 velocity=7
- added joint allegro_joint_11_tip: type fixed, parent link_11, child link_11_tip, origin xyz=0 0 0.026699999999999998 rpy=0 0 0
- added joint allegro_joint_12: type revolute, parent palm_link, child link_12, origin xyz=-0.0182 -0.019333 -0.045987 rpy=0 -1.6580627884499999 1.5707963259, axis +1 0 0, limit lower=0.263 upper=1.396 effort=15 velocity=7
- added joint allegro_joint_13: type revolute, parent link_12, child link_13, origin xyz=-0.027 -0.005 0.0399, axis 0 0 -1, limit lower=-0.10499999999999998 upper=1.1629999999999998 effort=15 velocity=7
- added joint allegro_joint_14: type revolute, parent link_13, child link_14, origin xyz=0 0 0.0177, axis 0 1 0, limit lower=-0.18899999999999997 upper=1.644 effort=15 velocity=7
- added joint allegro_joint_15: type revolute, parent link_14, child link_15, origin xyz=0 0 0.0514, axis 0 1 0, limit lower=-0.162 upper=1.7189999999999999 effort=15 velocity=7
- added joint allegro_joint_15_tip: type fixed, parent link_15, child link_15_tip, origin xyz=0 0 0.042300000000000004 rpy=0 0 0
- added joint allegro_joint_2: type revolute, parent link_1, child link_2, origin xyz=0 0 0.054, axis 0 1 0, limit lower=-0.17400000000000002 upper=1.7089999999999999 effort=15 velocity=7
- added joint allegro_joint_3: type revolute, parent link_2, child link_3, origin xyz=0 0 0.0384, axis 0 1 0, limit lower=-0.227 upper=1.6179999999999999 effort=15 velocity=7
- added joint allegro_joint_3_tip: type fixed, parent link_3, child link_3_tip, origin xyz=0 0 0.026699999999999998 rpy=0 0 0
- added joint allegro_joint_4: type revolute, parent palm_link, child link_4, origin xyz=0 0 0.0007 rpy=0.0 0 0, axis 0 0 1, limit lower=-0.47 upper=0.47 effort=15 velocity=7
- added joint allegro_joint_5: type revolute, parent link_4, child link_5, origin xyz=0 0 0.0164, axis 0 1 0, limit lower=-0.19599999999999998 upper=1.6099999999999999 effort=15 velocity=7
- added joint allegro_joint_6: type revolute, parent link_5, child link_6, origin xyz=0 0 0.054, axis 0 1 0, limit lower=-0.17400000000000002 upper=1.7089999999999999 effort=15 velocity=7
- added joint allegro_joint_7: type revolute, parent link_6, child link_7, origin xyz=0 0 0.0384, axis 0 1 0, limit lower=-0.227 upper=1.6179999999999999 effort=15 velocity=7
- added joint allegro_joint_7_tip: type fixed, parent link_7, child link_7_tip, origin xyz=0 0 0.026699999999999998 rpy=0 0 0
- added joint allegro_joint_8: type revolute, parent palm_link, child link_8, origin xyz=0 0.0435 -0.001542 rpy=-0.08726646254999999 0 0, axis 0 0 1, limit lower=-0.47 upper=0.47 effort=15 velocity=7
- added joint allegro_joint_9: type revolute, parent link_8, child link_9, origin xyz=0 0 0.0164, axis 0 1 0, limit lower=-0.19599999999999998 upper=1.6099999999999999 effort=15 velocity=7

File: ros2_source/src/allegro_hand_description/urdf/allegro_hand_description_right.urdf (robot description, URDF)
Before this commit: robot allegro_hand_right, 22 links, 21 joints
Joints:
- removed joint joint_0.0
- removed joint joint_1.0
- removed joint joint_10.0
- removed joint joint_11.0
- removed joint joint_11_tip
- removed joint joint_12.0
- removed joint joint_13.0
- removed joint joint_14.0
- removed joint joint_15.0
- removed joint joint_15_tip
- removed joint joint_2.0
- removed joint joint_3.0
- removed joint joint_3_tip
- removed joint joint_4.0
- removed joint joint_5.0
- removed joint joint_6.0
- removed joint joint_7.0
- removed joint joint_7_tip
- removed joint joint_8.0
- removed joint joint_9.0
- added joint allegro_joint_0.0: type revolute, parent palm_link, child link_0, origin xyz=0 0.0435 0 rpy=-0.08726646254999999 0 0, axis 0 0 1, limit lower=-0.47 upper=0.47 effort=15 velocity=7
- added joint allegro_joint_1.0: type revolute, parent link_0, child link_1, origin xyz=0 0 0.0164, axis 0 1 0, limit lower=-0.19599999999999998 upper=1.6099999999999999 effort=15 velocity=7
- added joint allegro_joint_10.0: type revolute, parent link_9, child link_10, origin xyz=0 0 0.054, axis 0 1 0, limit lower=-0.17400000000000002 upper=1.7089999999999999 effort=15 velocity=7
- added joint allegro_joint_11.0: type revolute, parent link_10, child link_11, origin xyz=0 0 0.0384, axis 0 1 0, limit lower=-0.227 upper=1.6179999999999999 effort=15 velocity=7
- added joint allegro_joint_11_tip: type fixed, parent link_11, child link_11_tip, origin xyz=0 0 0.026699999999999998 rpy=0 0 0
- added joint allegro_joint_12.0: type revolute, parent palm_link, child link_12, origin xyz=-0.0182 0.019333 -0.045987 rpy=0 -1.6580627884499999 -1.5707963259, axis -1 0 0, limit lower=0.263 upper=1.396 effort=15 velocity=7
- added joint allegro_joint_13.0: type revolute, parent link_12, child link_13, origin xyz=-0.027 0.005 0.0399, axis 0 0 1, limit lower=-0.10499999999999998 upper=1.1629999999999998 effort=15 velocity=7
- added joint allegro_joint_14.0: type revolute, parent link_13, child link_14, origin xyz=0 0 0.0177, axis 0 1 0, limit lower=-0.18899999999999997 upper=1.644 effort=15 velocity=7
- added joint allegro_joint_15.0: type revolute, parent link_14, child link_15, origin xyz=0 0 0.0514, axis 0 1 0, limit lower=-0.162 upper=1.7189999999999999 effort=15 velocity=7
- added joint allegro_joint_15_tip: type fixed, parent link_15, child link_15_tip, origin xyz=0 0 0.026699999999999998 rpy=0 0 0
- added joint allegro_joint_2.0: type revolute, parent link_1, child link_2, origin xyz=0 0 0.054, axis 0 1 0, limit lower=-0.17400000000000002 upper=1.7089999999999999 effort=15 velocity=7
- added joint allegro_joint_3.0: type revolute, parent link_2, child link_3, origin xyz=0 0 0.0384, axis 0 1 0, limit lower=-0.227 upper=1.6179999999999999 effort=15 velocity=7
- added joint allegro_joint_3_tip: type fixed, parent link_3, child link_3_tip, origin xyz=0 0 0.026699999999999998 rpy=0 0 0
- added joint allegro_joint_4.0: type revolute, parent palm_link, child link_4, origin xyz=0 0 0 rpy=0.0 0 0, axis 0 0 1, limit lower=-0.47 upper=0.47 effort=15 velocity=7
- added joint allegro_joint_5.0: type revolute, parent link_4, child link_5, origin xyz=0 0 0.0164, axis 0 1 0, limit lower=-0.19599999999999998 upper=1.6099999999999999 effort=15 velocity=7
- added joint allegro_joint_6.0: type revolute, parent link_5, child link_6, origin xyz=0 0 0.054, axis 0 1 0, limit lower=-0.17400000000000002 upper=1.7089999999999999 effort=15 velocity=7
- added joint allegro_joint_7.0: type revolute, parent link_6, child link_7, origin xyz=0 0 0.0384, axis 0 1 0, limit lower=-0.227 upper=1.6179999999999999 effort=15 velocity=7
- added joint allegro_joint_7_tip: type fixed, parent link_7, child link_7_tip, origin xyz=0 0 0.026699999999999998 rpy=0 0 0
- added joint allegro_joint_8.0: type revolute, parent palm_link, child link_8, origin xyz=0 -0.0435 0 rpy=0.08726646254999999 0 0, axis 0 0 1, limit lower=-0.47 upper=0.47 effort=15 velocity=7
- added joint allegro_joint_9.0: type revolute, parent link_8, child link_9, origin xyz=0 0 0.0164, axis 0 1 0, limit lower=-0.19599999999999998 upper=1.6099999999999999 effort=15 velocity=7

File: ros2_source/src/allegro_hand_description/urdf/allegro_hand_description_right_meta.urdf (robot description, URDF)
Before this commit: robot allegro_hand_right, 26 links, 25 joints
Joints:
- removed joint joint_0.0
- removed joint joint_1.0
- removed joint joint_10.0
- removed joint joint_11.0
- removed joint joint_12.0
- removed joint joint_13.0
- removed joint joint_14.0
- removed joint joint_15.0
- removed joint joint_2.0
- removed joint joint_3.0
- removed joint joint_4.0
- removed joint joint_5.0
- removed joint joint_6.0
- removed joint joint_7.0
- removed joint joint_8.0
- removed joint joint_9.0
- added joint allegro_joint_0.0: type revolute, parent palm_link, child link_0, origin xyz=0 0.0435 0 rpy=-0.08726646254999999 0 0, axis 0 0 1, limit lower=-0.47 upper=0.47 effort=15 velocity=7
- added joint allegro_joint_1.0: type revolute, parent link_0, child link_1, origin xyz=0 0 0.0164, axis 0 1 0, limit lower=-0.19599999999999998 upper=1.6099999999999999 effort=15 velocity=7
- added joint allegro_joint_10.0: type revolute, parent link_9, child link_10, origin xyz=0 0 0.054, axis 0 1 0, limit lower=-0.17400000000000002 upper=1.7089999999999999 effort=15 velocity=7
- added joint allegro_joint_11.0: type revolute, parent link_10, child link_11, origin xyz=0 0 0.0384, axis 0 1 0, limit lower=-0.227 upper=1.6179999999999999 effort=15 velocity=7
- added joint allegro_joint_12.0: type revolute, parent palm_link, child link_12, origin xyz=-0.0182 0.019333 -0.045987 rpy=0 -1.6580627884499999 -1.5707963259, axis -1 0 0, limit lower=0.263 upper=1.396 effort=15 velocity=7
- added joint allegro_joint_13.0: type revolute, parent link_12, child link_13, origin xyz=-0.027 0.005 0.0399, axis 0 0 1, limit lower=-0.10499999999999998 upper=1.1629999999999998 effort=15 velocity=7
- added joint allegro_joint_14.0: type revolute, parent link_13, child link_14, origin xyz=0 0 0.0177, axis 0 1 0, limit lower=-0.18899999999999997 upper=1.644 effort=15 velocity=7
- added joint allegro_joint_15.0: type revolute, parent link_14, child link_15, origin xyz=0 0 0.0514, axis 0 1 0, limit lower=-0.162 upper=1.7189999999999999 effort=15 velocity=7
- added joint allegro_joint_2.0: type revolute, parent link_1, child link_2, origin xyz=0 0 0.054, axis 0 1 0, limit lower=-0.17400000000000002 upper=1.7089999999999999 effort=15 velocity=7
- added joint allegro_joint_3.0: type revolute, parent link_2, child link_3, origin xyz=0 0 0.0384, axis 0 1 0, limit lower=-0.227 upper=1.6179999999999999 effort=15 velocity=7
- added joint allegro_joint_4.0: type revolute, parent palm_link, child link_4, origin xyz=0 0 0 rpy=0.0 0 0, axis 0 0 1, limit lower=-0.47 upper=0.47 effort=15 velocity=7
- added joint allegro_joint_5.0: type revolute, parent link_4, child link_5, origin xyz=0 0 0.0164, axis 0 1 0, limit lower=-0.19599999999999998 upper=1.6099999999999999 effort=15 velocity=7
- added joint allegro_joint_6.0: type revolute, parent link_5, child link_6, origin xyz=0 0 0.054, axis 0 1 0, limit lower=-0.17400000000000002 upper=1.7089999999999999 effort=15 velocity=7
- added joint allegro_joint_7.0: type revolute, parent link_6, child link_7, origin xyz=0 0 0.0384, axis 0 1 0, limit lower=-0.227 upper=1.6179999999999999 effort=15 velocity=7
- added joint allegro_joint_8.0: type revolute, parent palm_link, child link_8, origin xyz=0 -0.0435 0 rpy=0.08726646254999999 0 0, axis 0 0 1, limit lower=-0.47 upper=0.47 effort=15 velocity=7
- added joint allegro_joint_9.0: type revolute, parent link_8, child link_9, origin xyz=0 0 0.0164, axis 0 1 0, limit lower=-0.19599999999999998 upper=1.6099999999999999 effort=15 velocity=7
