Commit message: use link_12.0_left.obj

File: ros_source/src/allegro_hand_description/allegro_hand_description_left.urdf (robot description, URDF)
Before this commit: robot allegro_hand_left, 21 links, 20 joints
Links:
- link link_12.0: geometry collision box size=0.0358 0.034 0.0455; visual mesh filename=package://allegro_hand_description/meshes/link_12.0_left.obj
